File: 5way_cv_module/5way_cv_module.kicad_pcb (KiCad board)
At the start: 2 copper layers, 0 parts

Commit message: added opamp buffer better layout
Parts:
- added C1: 10uF, Capacitor_SMD:C_0603_1608Metric, F.Cu at (151.7, 46.4)
- added C2: 10uF, Capacitor_SMD:C_0603_1608Metric, F.Cu at (156.9, 42.1)
- added C3: 10uF, Capacitor_SMD:C_0603_1608Metric, F.Cu at (157.7, 52.1)
- added D1: LL4148, Diode_SMD:D_MiniMELF, F.Cu at (152.6, 50.1)
- added J1: I/O connector, cycfi_library:pin_header_1x3p_2.54mm_smd_horizontal, F.Cu at (152.7, 54.4)
- added J2: 5-way Switch Connector, cycfi_library:pin_socket_1x4p_2.54mm_smd_horizontal, B.Cu at (158.5, 58.8)
- added R1: 30k, Resistor_SMD:R_0402_1005Metric, F.Cu at (155.5, 49.1)
- added R2: 30k, Resistor_SMD:R_0402_1005Metric, F.Cu at (158.2, 49.1)
- added R3: 15k, Resistor_SMD:R_0402_1005Metric, F.Cu at (155.5, 50.4)
- added R4: 15k, Resistor_SMD:R_0402_1005Metric, F.Cu at (158.2, 50.4)
- added U1: HT7550-1, Package_TO_SOT_SMD:SOT-89-3, F.Cu at (152.4, 42.2)
- added U2: opamp_dbv2, Package_TO_SOT_SMD:SOT-23-5, F.Cu at (157.0, 45.4)
Routing:
- net common: track 0.00 -> 18.6 mm, vias 0 -> 2
- net OUT: track 0.00 -> 15.7 mm, vias 0 -> 2
- net middle: track 0.00 -> 14.5 mm, vias 0 -> 1
- net neck: track 0.00 -> 12.8 mm, vias 0 -> 1
- net V+: track 0.00 -> 11.3 mm
- net 5v: track 0.00 -> 11.1 mm
- net bridge: track 0.00 -> 9.30 mm, vias 0 -> 1
- net GND: track 0.00 -> 5.79 mm, vias 0 -> 1
- net Net-(C1-Pad1): track 0.00 -> 4.72 mm
- added copper zone on B.Cu, net GND
- added copper zone on F.Cu, net GND
Other:
- board outline added: 10.2 x 22.1 mm
- board text added: "5way CV Module v3.0"
- board text added: "GND"
- board text added: "OUT"
- board text added: "V+"

Commit message: added logo
Parts:
- added G***: LOGO, cycfi_library:cycfi-logo-9mm, B.Cu at (154.7, 39.8)
