File: audio_buffer/audio_buffer.kicad_sch (KiCad schematic)
At the start: 13 parts, among them J1 conn_1x3, J2 conn_1x3, Q1 LBSS84LT1G, U1 OPA197IDBV

Commit message: Switch to triangular solder shunt
Parts:
- JP1: footprint Jumper:SolderJumper-2_P1.3mm_Open_RoundedPad1.0x1.5mm -> Jumper:SolderJumper-2_P1.3mm_Open_TrianglePad1.0x1.5mm
Changed lines of the file:
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@@
 			)
 		)
-		(property "Footprint" "Jumper:SolderJumper-2_P1.3mm_Open_RoundedPad1.0x1.5mm"
+		(property "Footprint" "Jumper:SolderJumper-2_P1.3mm_Open_TrianglePad1.0x1.5mm"
 			(at 179.07 111.76 0)
 			(effects
