File: audio_pot_big/audio_pot_big.kicad_pcb (KiCad board)
At the start: 2 copper layers, 24.2 x 18 mm, 16 parts, among them J1 Conn_02x03_Counter_Clockwise, Q1 LBSS84LT1G, U1 OPA197IDBV

Commit message: Schematics minor updates (net naming)
Connections:
- net /pot_wiper renamed Net-(C2-Pad2)
- net in+ renamed IN+
- net out renamed OUT
- net v+ renamed V+
- net vcc renamed VCC
Changed lines of the file:
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@@
 	(net 1 "/+IN")
 	(net 2 "GND")
-	(net 3 "vcc")
-	(net 4 "/pot_wiper")
-	(net 5 "/-IN")
-	(net 6 "Net-(JP3-A)")
-	(net 7 "out")
-	(net 8 "v+")
-	(net 9 "in+")
+	(net 3 "/-IN")
+	(net 4 "Net-(JP3-A)")
+	(net 5 "Net-(C2-Pad2)")
+	(net 6 "VCC")
+	(net 7 "OUT")
+	(net 8 "V+")
+	(net 9 "IN+")
 	(footprint "Resistor_SMD:R_0402_1005Metric"
 		(layer "F.Cu")
@@
 			(layers "F.Cu" "F.Mask" "F.Paste")
 			(roundrect_rratio 0.25)
-			(net 3 "vcc")
+			(net 6 "VCC")
 			(pintype "passive")
 		)
@@
 			(layers "F.Cu" "F.Mask" "F.Paste")
 			(roundrect_rratio 0.25)
-			(net 3 "vcc")
+			(net 6 "VCC")
 			(pinfunction "S")
 			(pintype "passive")
@@
 			(layers "F.Cu" "F.Mask" "F.Paste")
 			(roundrect_rratio 0.25)
-			(net 8 "v+")
+			(net 8 "V+")
 			(pinfunction "D")
 			(pintype "passive")
@@
 			(size 0.3 0.3)
 			(layers "F.Cu" "F.Mask")
-			(net 6 "Net-(JP3-A)")
+			(net 4 "Net-(JP3-A)")
 			(pinfunction "A")
 			(pintype "passive")
@@
 			(size 0.3 0.3)
 			(layers "F.Cu" "F.Mask")
-			(net 7 "out")
+			(net 7 "OUT")
 			(pinfunction "B")
 			(pintype "passive")
@@
 			(layers "F.Cu" "F.Mask" "F.Paste")
 			(roundrect_rratio 0.25)
-			(net 6 "Net-(JP3-A)")
+			(net 4 "Net-(JP3-A)")
 			(pintype "passive")
 		)
@@
 			(layers "F.Cu" "F.Mask" "F.Paste")
 			(roundrect_rratio 0.25)
-			(net 5 "/-IN")
+			(net 3 "/-IN")
 			(pintype "passive")
 		)
@@
 			(layers "*.Cu" "*.Mask")
 			(remove_unused_layers no)
-			(net 9 "in+")
+			(net 9 "IN+")
 			(pinfunction "1")
 			(pintype "passive")
@@
 			(layers "*.Cu" "*.Mask")
 			(remove_unused_layers no)
-			(net 4 "/pot_wiper")
+			(net 5 "Net-(C2-Pad2)")
 			(pinfunction "2")
 			(pintype "passive")
@@
 			(layers "F.Cu" "F.Mask" "F.Paste")
 			(roundrect_rratio 0.25)
-			(net 7 "out")
+			(net 7 "OUT")
 			(pintype "passive")
 		)
@@
 			(layers "F.Cu" "F.Mask" "F.Paste")
 			(roundrect_rratio 0.25)
-			(net 6 "Net-(JP3-A)")
+			(net 4 "Net-(JP3-A)")
 			(pintype "passive")
 		)
@@
 			(layers "F.Cu" "F.Mask" "F.Paste")
 			(roundrect_rratio 0.25)
-			(net 3 "vcc")
+			(net 6 "VCC")
 			(pintype "passive")
 		)
@@
 			(layers "F.Cu" "F.Mask" "F.Paste")
 			(roundrect_rratio 0.25)
-			(net 4 "/pot_wiper")
+			(net 5 "Net-(C2-Pad2)")
 			(pintype "passive")
 		)
@@
 			(layers "F.Cu" "F.Mask" "F.Paste")
 			(roundrect_rratio 0.25)
-			(net 3 "vcc")
+			(net 6 "VCC")
 			(pintype "passive")
 		)
@@
 			(layers "F.Cu" "F.Mask" "F.Paste")
 			(roundrect_rratio 0.25)
-			(net 6 "Net-(JP3-A)")
+			(net 4 "Net-(JP3-A)")
 			(pintype "passive")
 		)
@@
 			(layers "F.Cu" "F.Mask" "F.Paste")
 			(roundrect_rratio 0.25)
-			(net 5 "/-IN")
+			(net 3 "/-IN")
 			(pintype "output")
 		)
@@
 			(layers "F.Cu" "F.Mask" "F.Paste")
 			(roundrect_rratio 0.25)
-			(net 5 "/-IN")
+			(net 3 "/-IN")
 			(pinfunction "-")
 			(pintype "input")
@@
 			(layers "F.Cu" "F.Mask" "F.Paste")
 			(roundrect_rratio 0.25)
-			(net 3 "vcc")
+			(net 6 "VCC")
 			(pinfunction "V+")
 			(pintype "power_in")
@@
 			(size 3.17 1.02)
 			(layers "F.Cu" "F.Mask" "F.Paste")
-			(net 9 "in+")
+			(net 9 "IN+")
 			(pinfunction "Pin_1")
 			(pintype "passive")
@@
 			(size 3.17 1.02)
 			(layers "F.Cu" "F.Mask" "F.Paste")
-			(net 8 "v+")
+			(net 8 "V+")
 			(pinfunction "Pin_3")
 			(pintype "passive")
@@
 			(size 3.17 1.02)
 			(layers "F.Cu" "F.Mask" "F.Paste")
-			(net 8 "v+")
+			(net 8 "V+")
 			(pinfunction "Pin_4")
 			(pintype "passive")
@@
 			(size 3.17 1.02)
 			(layers "F.Cu" "F.Mask" "F.Paste")
-			(net 7 "out")
+			(net 7 "OUT")
 			(pinfunction "Pin_6")
 			(pintype "passive")
@@
 	)
 	(segment
-		(start 153.7075 84.26)
-		(end 153.7075 86.0425)
-		(width 0.6)
+		(start 143.6975 86.499999)
+		(end 144.023501 86.826)
+		(width 0.25)
 		(layer "F.Cu")
 		(net 3)
 	)
 	(segment
-		(start 143.6975 83.5625)
-		(end 143.6975 81.92)
-		(width 0.6)
+		(start 146.25 84.215)
+		(end 146.25 86.826)
+		(width 0.25)
 		(layer "F.Cu")
 		(net 3)
 	)
 	(segment
-		(start 153.7075 86.0425)
-		(end 151.55 88.2)
-		(width 0.6)
+		(start 145.5975 83.5625)
+		(end 146.25 84.215)
+		(width 0.25)
 		(layer "F.Cu")
 		(net 3)
 	)
 	(segment
-		(start 142.8965 86.62381)
-		(end 142.8965 84.3635)
-		(width 0.6)
+		(start 146.25 86.826)
+		(end 147.1715 86.826)
+		(width 0.25)
 		(layer "F.Cu")
 		(net 3)
 	)
 	(segment
-		(start 143.6975 83.5625)
-		(end 142.11 81.975)
-		(width 0.6)
+		(start 147.1715 86.826)
+		(end 147.4975 86.5)
+		(width 0.25)
 		(layer "F.Cu")
 		(net 3)
 	)
 	(segment
-		(start 155.8975 84.35)
-		(end 153.7975 84.35)
-		(width 0.6)
+		(start 143.6975 85.8375)
+		(end 143.6975 86.499999)
+		(width 0.25)
 		(layer "F.Cu")
 		(net 3)
 	)
 	(segment
-		(start 143.6975 81.92)
-		(end 143.7175 81.9)
-		(width 0.6)
+		(start 144.023501 86.826)
+		(end 146.25 86.826)
+		(width 0.25)
 		(layer "F.Cu")
 		(net 3)
 	)
 	(segment
-		(start 142.11 81.975)
-		(end 142.11 81.8)
-		(width 0.6)
+		(start 147.6475 82.0425)
+		(end 148.99 80.7)
+		(width 0.25)
 		(layer "F.Cu")
-		(net 3)
+		(net 4)
 	)
 	(segment
-		(start 144.47269 88.2)
-		(end 142.8965 86.62381)
-		(width 0.6)
+		(start 147.6475 83.8)
+		(end 147.6475 82.0425)
+		(width 0.25)
 		(layer "F.Cu")
-		(net 3)
+		(net 4)
 	)
 	(segment
-		(start 153.7975 84.35)
-		(end 153.7075 84.26)
-		(width 0.6)
+		(start 150.8975 85.99)
+		(end 149.9075 85.99)
+		(width 0.25)
 		(layer "F.Cu")
-		(net 3)
+		(net 4)
 	)
 	(segment
-		(start 142.8965 84.3635)
-		(end 143.6975 83.5625)
-		(width 0.6)
+		(start 149.3975 86.5)
+		(end 147.6475 84.75)
+		(width 0.25)
 		(layer "F.Cu")
-		(net 3)
+		(net 4)
 	)
 	(segment
-		(start 151.55 88.2)
-		(end 144.47269 88.2)
-		(width 0.6)
+		(start 149.9075 85.99)
+		(end 149.3975 86.5)
+		(width 0.25)
 		(layer "F.Cu")
-		(net 3)
+		(net 4)
+	)
+	(segment
+		(start 147.6475 84.75)
+		(end 147.6475 83.8)
+		(width 0.25)
+		(layer "F.Cu")
+		(net 4)
 	)
 	(segment
@@
 		(width 0.25)
 		(layer "F.Cu")
-		(net 4)
+		(net 5)
 	)
 	(segment
@@
 		(width 0.25)
 		(layer "F.Cu")
-		(net 4)
+		(net 5)
 	)
 	(segment
@@
 		(width 0.25)
 		(layer "F.Cu")
-		(net 4)
-	)
-	(segment
-		(start 143.6975 86.499999)
-		(end 144.023501 86.826)
-		(width 0.25)
-		(layer "F.Cu")
 		(net 5)
 	)
 	(segment
-		(start 146.25 84.215)
-		(end 146.25 86.826)
-		(width 0.25)
+		(start 153.7075 84.26)
+		(end 153.7075 86.0425)
+		(width 0.6)
 		(layer "F.Cu")
-		(net 5)
+		(net 6)
 	)
 	(segment
-		(start 145.5975 83.5625)
-		(end 146.25 84.215)
-		(width 0.25)
+		(start 143.6975 83.5625)
+		(end 143.6975 81.92)
+		(width 0.6)
 		(layer "F.Cu")
-		(net 5)
+		(net 6)
 	)
 	(segment
-		(start 146.25 86.826)
-		(end 147.1715 86.826)
-		(width 0.25)
+		(start 153.7075 86.0425)
+		(end 151.55 88.2)
+		(width 0.6)
 		(layer "F.Cu")
-		(net 5)
+		(net 6)
 	)
 	(segment
-		(start 147.1715 86.826)
-		(end 147.4975 86.5)
-		(width 0.25)
+		(start 142.8965 86.62381)
+		(end 142.8965 84.3635)
+		(width 0.6)
 		(layer "F.Cu")
-		(net 5)
+		(net 6)
 	)
 	(segment
-		(start 143.6975 85.8375)
-		(end 143.6975 86.499999)
-		(width 0.25)
+		(start 143.6975 83.5625)
+		(end 142.11 81.975)
+		(width 0.6)
 		(layer "F.Cu")
-		(net 5)
+		(net 6)
 	)
 	(segment
-		(start 144.023501 86.826)
-		(end 146.25 86.826)
-		(width 0.25)
+		(start 155.8975 84.35)
+		(end 153.7975 84.35)
+		(width 0.6)
 		(layer "F.Cu")
-		(net 5)
+		(net 6)
 	)
 	(segment
-		(start 147.6475 82.0425)
-		(end 148.99 80.7)
-		(width 0.25)
+		(start 143.6975 81.92)
+		(end 143.7175 81.9)
+		(width 0.6)
 		(layer "F.Cu")
 		(net 6)
 	)
 	(segment
-		(start 147.6475 83.8)
-		(end 147.6475 82.0425)
-		(width 0.25)
+		(start 142.11 81.975)
+		(end 142.11 81.8)
+		(width 0.6)
 		(layer "F.Cu")
 		(net 6)
 	)
 	(segment
-		(start 150.8975 85.99)
-		(end 149.9075 85.99)
-		(width 0.25)
+		(start 144.47269 88.2)
+		(end 142.8965 86.62381)
+		(width 0.6)
 		(layer "F.Cu")
 		(net 6)
 	)
 	(segment
-		(start 149.3975 86.5)
-		(end 147.6475 84.75)
-		(width 0.25)
+		(start 153.7975 84.35)
+		(end 153.7075 84.26)
+		(width 0.6)
 		(layer "F.Cu")
 		(net 6)
 	)
 	(segment
-		(start 149.9075 85.99)
-		(end 149.3975 86.5)
-		(width 0.25)
+		(start 142.8965 84.3635)
+		(end 143.6975 83.5625)
+		(width 0.6)
 		(layer "F.Cu")
 		(net 6)
 	)
 	(segment
-		(start 147.6475 84.75)
-		(end 147.6475 83.8)
-		(width 0.25)
+		(start 151.55 88.2)
+		(end 144.47269 88.2)
+		(width 0.6)
 		(layer "F.Cu")
 		(net 6)
