File: audio_pot_big/audio_pot_big.kicad_sch (KiCad schematic)
At the start: 15 parts, among them J1 Conn_02x03_Counter_Clockwise, Q1 LBSS84LT1G, U1 OPA197IDBV

Commit message: Schematics minor updates (net naming)
Connections:
- net in+ renamed IN+
- net out renamed OUT
- net v+ renamed V+
- net vcc renamed VCC
Other:
- moved on the sheet: C2
Changed lines of the file:
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@@
 	(wire
 		(pts
-			(xy 108.585 114.935) (xy 111.125 114.935)
+			(xy 105.41 114.935) (xy 111.125 114.935)
 		)
 		(stroke
@@
 	(wire
 		(pts
-			(xy 92.075 114.935) (xy 100.965 114.935)
+			(xy 92.075 114.935) (xy 97.79 114.935)
 		)
 		(stroke
@@
 		)
 	)
-	(global_label "in+"
+	(global_label "IN+"
 		(shape input)
 		(at 84.455 94.615 180)
@@
 		)
 	)
-	(global_label "in+"
+	(global_label "IN+"
 		(shape input)
 		(at 83.185 54.61 180)
@@
 		)
 	)
-	(global_label "out"
+	(global_label "OUT"
 		(shape input)
 		(at 190.5 117.475 0)
@@
 		)
 	)
-	(global_label "vcc"
+	(global_label "VCC"
 		(shape input)
 		(at 106.045 94.615 180)
@@
 		)
 	)
-	(global_label "v+"
+	(global_label "V+"
 		(shape input)
 		(at 95.885 59.69 0)
@@
 		)
 	)
-	(global_label "vcc"
+	(global_label "VCC"
 		(shape input)
 		(at 134.62 106.045 0)
@@
 		)
 	)
-	(global_label "vcc"
+	(global_label "VCC"
 		(shape input)
 		(at 195.58 50.8 0)
@@
 		)
 	)
-	(global_label "v+"
+	(global_label "V+"
 		(shape input)
 		(at 153.67 50.8 180)
@@
 		)
 	)
-	(global_label "out"
+	(global_label "OUT"
 		(shape input)
 		(at 95.885 54.61 0)
@@
 		)
 	)
-	(global_label "v+"
+	(global_label "V+"
 		(shape input)
 		(at 83.185 59.69 180)
@@
 	(symbol
 		(lib_id "Device:C")
-		(at 104.775 114.935 270)
+		(at 101.6 114.935 270)
 		(unit 1)
 		(exclude_from_sim no)
@@
 		(dnp no)
 		(property "Reference" "C2"
-			(at 104.775 108.5342 90)
+			(at 101.6 108.5342 90)
 			(effects
 				(font
@@
 		)
 		(property "Value" "100nF"
-			(at 104.775 110.8456 90)
+			(at 101.6 110.8456 90)
 			(effects
 				(font
@@
 		)
 		(property "Footprint" "Capacitor_SMD:C_0805_2012Metric"
-			(at 100.965 115.9002 0)
+			(at 97.79 115.9002 0)
 			(effects
 				(font
@@
 		)
 		(property "Datasheet" "~"
-			(at 104.775 114.935 0)
-			(effects
-				(font
-					(size 1.27 1.27)
-				)
-				(hide yes)
-			)
-		)
-		(property "Description" ""
-			(at 104.775 114.935 0)
+			(at 101.6 114.935 0)
+			(effects
+				(font
+					(size 1.27 1.27)
+				)
+				(hide yes)
+			)
+		)
+		(property "Description" ""
+			(at 101.6 114.935 0)
 			(effects
 				(font
@@
 		)
 		(property "LCSC" "C49678"
-			(at 104.775 114.935 0)
-			(effects
-				(font
+			(at 101.6 114.935 0)
+			(effects
+				(font

Commit message: - Fab updates - Added SMD 2x3P header
Parts:
- H1, H2, RV1: now left out of the parts list
- J1: JLCPCB_CORRECTION (none) -> 0;0;90; LCSC (none) -> C46061685
- U1: JLCPCB_CORRECTION 0;0;270 -> 0;0;180
Changed lines of the file:
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@@
 			)
 		)
-		(property "JLCPCB_CORRECTION" "0;0;270"
+		(property "JLCPCB_CORRECTION" "0;0;180"
 			(at 133.35 117.475 0)
 			(effects
@@
 				(font
 					(size 1.27 1.27)
+				)
+				(hide yes)
+			)
+		)
+		(property "LCSC" "C46061685"
+			(at 88.265 57.15 0)
+			(effects
+				(font
+					(size 1.524 1.524)
+				)
+				(hide yes)
+			)
+		)
+		(property "JLCPCB_CORRECTION" "0;0;90"
+			(at 88.265 57.15 0)
+			(effects
+				(font
+					(size 1.524 1.524)
 				)
 				(hide yes)
@@
 		(unit 1)
 		(exclude_from_sim no)
-		(in_bom yes)
+		(in_bom no)
 		(on_board yes)
 		(dnp no)
@@
 		(unit 1)
 		(exclude_from_sim no)
-		(in_bom yes)
+		(in_bom no)
 		(on_board yes)
 		(dnp no)
@@
 		(unit 1)
 		(exclude_from_sim no)
-		(in_bom yes)
-		(on_board yes)
-		(dnp no)
+		(in_bom no)
+		(on_board yes)
+		(dnp no)
